Commit message: Rebase from 'upstream'

File: webots_ros2_importer/webots_ros2_importer/urdf2webots/tests/sources/kuka_lbr_iiwa_support/urdf/model.urdf (robot description, URDF)
Before this commit: robot kuka_lbr_iiwa_14_r820, 10 links, 9 joints
Joints:
- joint base_link-base: child base -> base_link; parent base_link -> base
