Commit message: Rebase from 'upstream'

File: webots_ros2_importer/webots_ros2_importer/urdf2webots/tests/sources/gait2392_simbody/urdf/human.urdf (robot description, URDF)
Before this commit: robot human, 20 links, 19 joints
Links:
- link calcn_r: geometry collision mesh filename=../meshes/obj/Calcn L.001.obj scale=1.0 -1.0 1.0; visual mesh filename=../meshes/obj/Calcn L.obj scale=1.0 -1.0 1.0

File: webots_ros2_importer/webots_ros2_importer/urdf2webots/tests/sources/kuka_lbr_iiwa_support/urdf/model.urdf (robot description, URDF)
Before this commit: robot kuka_lbr_iiwa_14_r820, 10 links, 9 joints
Links:
- link link_5: geometry collision mesh filename=package://kuka_lbr_iiwa_support/meshes/lbr_iiwa_14_r820/col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; visual mesh filename=package://kuka_lbr_iiwa_support/meshes/lbr_iiwa_14_r820/vis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 scale=-1.0 -1.0 -1.0

Commit message: Rebase from 'upstream'

File: webots_ros2_importer/webots_ros2_importer/urdf2webots/tests/sources/gait2392_simbody/urdf/human.urdf (robot description, URDF)
Before this commit: robot human, 20 links, 19 joints
Links:
- link calcn_r: geometry collision mesh filename=../meshes/obj/Calcn R.001.obj scale=1.0 1.0 1.0; visual mesh filename=../meshes/obj/Calcn L.obj scale=1.0 -1.0 1.0

File: webots_ros2_universal_robot/resource/Universal_Robots_ROS2_Driver/ur_description/urdf/inc/ur_common.xacro (robot description, xacro)
@@ -22,8 +22,8 @@
   <xacro:macro name="read_model_data" params="joint_limits_parameters_file kinematics_parameters_file physical_parameters_file visual_parameters_file">
     <!-- Read .yaml files from disk, load content into properties -->
-    <xacro:property name="config_joint_limit_parameters" value="${load_yaml(joint_limits_parameters_file)}"/>
-    <xacro:property name="config_kinematics_parameters" value="${load_yaml(kinematics_parameters_file)}"/>
-    <xacro:property name="config_physical_parameters" value="${load_yaml(physical_parameters_file)}"/>
-    <xacro:property name="config_visual_parameters" value="${load_yaml(visual_parameters_file)}"/>
+    <xacro:property name="config_joint_limit_parameters" value="${xacro.load_yaml(joint_limits_parameters_file)}"/>
+    <xacro:property name="config_kinematics_parameters" value="${xacro.load_yaml(kinematics_parameters_file)}"/>
+    <xacro:property name="config_physical_parameters" value="${xacro.load_yaml(physical_parameters_file)}"/>
+    <xacro:property name="config_visual_parameters" value="${xacro.load_yaml(visual_parameters_file)}"/>
     <!-- Extract subsections from yaml dictionaries -->
     <xacro:property name="sec_limits" value="${config_joint_limit_parameters['joint_limits']}"/>

File: webots_ros2_universal_robot/resource/Universal_Robots_ROS2_Driver/ur_description/urdf/ur.urdf.xacro (robot description, xacro)
@@ -38,5 +38,5 @@
      fake_sensor_commands="$(arg fake_sensor_commands)"
      headless_mode="$(arg headless_mode)"
-     initial_positions="${load_yaml(initial_positions_file)}"
+     initial_positions="${xacro.load_yaml(initial_positions_file)}"
      use_tool_communication="$(arg use_tool_communication)" />
 </robot>
